Commit message: chore: rename workshop to ossna 26
Renames the workshop materials, package, docker image, and docs
from roscon-25-workshop to ossna-26-workshop.

File: px4_ossna_26/px4_ossna_26/urdf/x500.urdf (robot description, URDF)
Before this commit: robot x500, 5 links, 4 joints
Links:
- link base_link: geometry visual mesh filename=package://px4_ossna_26/meshes/5010Base.dae; visual mesh filename=package://px4_ossna_26/meshes/5010Base.dae
- link motor_0: geometry visual mesh filename=package://px4_ossna_26/meshes/5010Bell.dae
- link motor_1: geometry visual mesh filename=package://px4_ossna_26/meshes/5010Bell.dae
- link motor_2: geometry visual mesh filename=package://px4_ossna_26/meshes/5010Bell.dae
- link motor_3: geometry visual mesh filename=package://px4_ossna_26/meshes/5010Bell.dae
